Commit message: pushing basic ball catching code

File: three_link.urdf (robot description, URDF)
Before this commit: robot three_link_robot, 4 links, 3 joints
Links:
- added link end_effector, mass 0.0; visual box size=0.02 0.02 0.02
- link arm1: mass 0.0754 -> 0.07539822368615504
- link arm2: mass 0.0754 -> 0.07539822368615504
- link arm3: mass 0.0754 -> 0.07539822368615504
Joints:
- added joint end_effector_on_end: type fixed, parent arm3, child end_effector, origin xyz=0.2 0 0 rpy=0 0 0
